File: PCB/Buttons.kicad_sch (KiCad schematic)
At the start: 40 parts

Commit message: v1.0
Parts:
- MX10, MX12, MX14, MX15, MX17, MX19, MX2, MX21, MX23, MX26, MX28, MX29, MX32, MX33, MX36, MX38, MX39, MX4, MX5, MX8: now left out of the parts list
Other:
- moved on the sheet: MX1, MX10, MX2, MX27, MX28, MX29, MX3, MX30, MX4, MX5, MX6, MX7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
