File: PCB/IntegratedOF1.kicad_pcb (KiCad board)
At the start: 2 copper layers, 347 x 156.5 mm, 81 parts, among them J1 USB C Connector, J2 JTAG_TC2030, J3 Conn_01x02_Pin, SW1 Boot, U1 XC6206, U2 USBLC6-2SC6, U3 RP2040, U4 W25Q128JVS, Y1 12MHz

Commit message: Adjusted PCB and BOM
- Adjusted PCB to add missing screw hole and repositioned one more according to the plate file.
- Move the shield resistor to a new position where it shouldn't interfere with some cases.
- Added a new cutout in the PCB so it's easier to extract from a F1 case.
- Changed Schottky diode and boot button part # so they use a basic part instead of an extended one.
Parts:
- moved R1 3.70 mm to (212.6, 29.2)
Routing:
- net Net-(J1-SHIELD): track 26.8 -> 24.0 mm
- net GND: track 50.2 -> 51.5 mm, vias 14 -> 15
Other:
- outline, holes or cut-outs redrawn
