File: PCB/IntegratedOF1.kicad_sch (KiCad schematic)
At the start: 42 parts, among them J1 USB C Connector, J2 JTAG_TC2030, J3 Conn_01x02_Pin, SW1 Boot, U1 XC6206, U2 USBLC6-2SC6, U3 RP2040, U4 W25Q128JVS, Y1 12MHz

Commit message: Adjusted PCB and BOM
- Adjusted PCB to add missing screw hole and repositioned one more according to the plate file.
- Move the shield resistor to a new position where it shouldn't interfere with some cases.
- Added a new cutout in the PCB so it's easier to extract from a F1 case.
- Changed Schottky diode and boot button part # so they use a basic part instead of an extended one.
Parts:
- D1, D2: LCSC C130880 -> C8598
Changed lines of the file:
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@@
       (effects (font (size 1.27 1.27)) hide)
     )
-    (property "LCSC" "C130880" (at 209.55 108.204 0)
+    (property "LCSC" "C8598" (at 209.55 108.204 0)
       (effects (font (size 1.27 1.27)) hide)
     )
@@
       (effects (font (size 1.27 1.27)) hide)
     )
-    (property "LCSC" "C130880" (at 171.45 87.63 0)
-      (effects (font (size 1.27 1.27)) hide)
-    )
+    (property "LCSC" "C8598" (at 171.45 87.63 0)
+      (effects (font (size 1.27 1.27)) hide)
+    )

Commit message: v1.0
Parts:
- D3: LCSC (none) -> C2297
- F1: LCSC (none) -> C2836286
- J2, J3: now left out of the parts list
- R1: LCSC C25190 -> C22935
- R2, R3: LCSC C25744 -> C25905
- R4: LCSC (none) -> C25117
- R5: LCSC (none) -> C23189
- R6: LCSC (none) -> C25804
- SW1: now in the parts list
- U2: LCSC (none) -> C2827654
Changed lines of the file:
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@@
   )
   (symbol (lib_id "Connector:Conn_01x02_Pin") (at 110.49 119.634 270) (unit 1)
-    (in_bom yes) (on_board yes) (dnp no) (fields_autoplaced)
+    (in_bom no) (on_board yes) (dnp no) (fields_autoplaced)
     (property "Reference" "J3" (at 111.506 120.904 90)
       (effects (font (size 1.27 1.27)) (justify left))
@@
       (effects (font (size 1.27 1.27)) hide)
     )
-    (property "LCSC" "C25190" (at 101.6 28.956 0)
+    (property "LCSC" "C22935" (at 101.6 28.956 0)
       (effects (font (size 1.27 1.27)) hide)
     )
@@
       (effects (font (size 1.27 1.27)) hide)
     )
+    (property "LCSC" "C25117" (at 208.9658 132.588 90)
+      (effects (font (size 1.27 1.27)) hide)
+    )
     (pin "1")
     (pin "2")
@@
       (effects (font (size 1.27 1.27)) hide)
     )
+    (property "LCSC" "C23189" (at 200.66 157.48 90)
+      (effects (font (size 1.27 1.27)) hide)
+    )
     (pin "1")
     (pin "2")
@@
       (effects (font (size 1.27 1.27)) hide)
     )
+    (property "LCSC" "C2836286" (at 170.18 54.356 90)
+      (effects (font (size 1.27 1.27)) hide)
+    )
     (pin "1")
     (pin "2")
@@
   )
   (symbol (lib_id "marbastlib-various:JTAG_TC2030") (at 162.052 180.086 0) (unit 1)
-    (in_bom yes) (on_board yes) (dnp no)
+    (in_bom no) (on_board yes) (dnp no)
     (property "Reference" "J2" (at 169.3418 177.5459 0)
       (effects (font (size 1.27 1.27)) (justify left))
@@
       (effects (font (size 1.27 1.27)) hide)
     )
-    (property "LCSC" "C25744" (at 162.56 54.356 0)
+    (property "LCSC" "C25905" (at 162.56 54.356 0)
       (effects (font (size 1.27 1.27)) hide)
     )
@@
   )
   (symbol (lib_id "Switch:SW_Push") (at 109.347 134.874 0) (unit 1)
-    (in_bom no) (on_board yes) (dnp no) (fields_autoplaced)
+    (in_bom yes) (on_board yes) (dnp no) (fields_autoplaced)
     (property "Reference" "SW1" (at 109.347 128.27 0)
       (effects (font (size 1.27 1.27)))
@@
       (effects (font (size 1.27 1.27)) hide)
     )
-    (property "LCSC" "C25744" (at 165.1 54.356 0)
+    (property "LCSC" "C25905" (at 165.1 54.356 0)
       (effects (font (size 1.27 1.27)) hide)
     )
@@
       (effects (font (size 1.27 1.27)) hide)
     )
+    (property "LCSC" "C2297" (at 214.0458 132.588 0)
+      (effects (font (size 1.27 1.27)) hide)
+    )
     (pin "1")
     (pin "2")
@@
       (effects (font (size 1.27 1.27)) hide)
     )
+    (property "LCSC" "C25804" (at 208.4578 157.48 90)
+      (effects (font (size 1.27 1.27)) hide)
+    )
     (pin "1")
     (pin "2")
@@
       (effects (font (size 1.27 1.27)) hide)
     )
+    (property "LCSC" "C2827654" (at 117.602 90.932 0)
+      (effects (font (size 1.27 1.27)) hide)
+    )

Commit message: Adjusted push button to the correct part number
Parts:
- SW1: LCSC C5156480 -> C318884
Changed lines of the file:
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@@
       (effects (font (size 1.27 1.27)) hide)
     )
-    (property "LCSC" "C5156480" (at 109.347 134.874 0)
+    (property "LCSC" "C318884" (at 109.347 134.874 0)
       (effects (font (size 1.27 1.27)) hide)
     )
